File: know.kicad_sch (KiCad schematic)
At the start: 23 parts, among them U1 OPA380AIDGKT, U2 OPA2320AID, U3 LMP7721MA_NOPB, U4 TLV333IDBVT, U5 DAC7571IDBVT, U6 OPA2320AID

Commit message: Add files via upload
Parts:
- removed U1: OPA380AIDGKT, OPA380AIDGKT:SOP65P490X110-8N, symbol OPA380AIDGKT:OPA380AIDGKT
- removed U2, U6: OPA2320AID, OPA2320AID:SOIC127P599X175-8N, symbol OPA2320AID:OPA2320AID
- removed U3: LMP7721MA_NOPB, LMP7721MA_NOPB:SOIC127P599X175-8N, symbol LMP7721MA_NOPB:LMP7721MA_NOPB
- removed U4: TLV333IDBVT, TLV333IDBVT:SOT95P280X145-5N, symbol TLV333IDBVT:TLV333IDBVT
- removed U5: DAC7571IDBVT, DAC7571IDBVT:SOT95P280X145-6N, symbol DAC7571IDBVT:DAC7571IDBVT
- added DAC7571: DAC7571IDBVT, DAC7571:SOT95P280X145-6N, symbol DAC7571IDBVT:DAC7571IDBVT
- added JWF1: TS5A4624DCKR, JWF:DCK6, symbol 2026-04-15_06-22-13:TS5A4624DCKR
- added LMP7721: LMP7721MA_NOPB, lmp7721:SOIC127P599X175-8N, symbol LMP7721MA_NOPB:LMP7721MA_NOPB
- added OPA2320_1, OPA2320_2: OPA2320AID, opa2320:SOIC127P599X175-8N, symbol OPA2320AID:OPA2320AID
- added OSD5-5D1: OSD5-5D, Package_TO_SOT_THT:TO-5-2, symbol Device:D_Photo
- added R10: R_US, Resistor_SMD:R_0603_1608Metric, symbol Device:R_US
- added R11: R, Resistor_SMD:R_0201_0603Metric, symbol Device:R
- added TLV333: TLV333IDBVT, TLV333:SOT95P280X145-5N, symbol TLV333IDBVT:TLV333IDBVT
- C1, C2, C3, C4, C5, C6, C7, C8: footprint (none) -> Capacitor_SMD:C_0603_1608Metric
- R1, R2, R3, R4, R5, R6, R7, R8, R9: footprint (none) -> Resistor_SMD:R_0603_1608Metric
Connections:
- net 2320_1_1: now also JWF1.4 (NC), OPA2320_1.1 (VOUTA)
- net 2320_1_2: now also OPA2320_1.2 (-INA)
- net 2320_1_6: now also OPA2320_1.6 (-INB)
- net 2320_1_7: now also JWF1.6 (NO), OPA2320_1.7 (VOUTB)
- net 2320_2_1: now also OPA2320_2.1 (VOUTA), OPA2320_2.2 (-INA), TLV333.3 (+IN)
- net 2320_2_3: now also OPA2320_2.3 (+INA), R10.2
- net 2320_2_5: now also OPA2320_2.5 (+INB), TLV333.1 (OUT)
- net 2320_2_6: now also OPA2320_2.6 (-INB)
- net 2320_2_7: now also OPA2320_2.7 (VOUTB)
- net 2320_2_8: now also OPA2320_1.8 (V+), OPA2320_2.8 (V+)
- net 333_4: now also DAC7571.1 (VOUT), TLV333.4 (-IN)
- net 7721_1: now also LMP7721.1
- net 7721_4: now also LMP7721.4, LMP7721.6, TLV333.5 (V+)
- net GND: now also DAC7571.2 (GND), JWF1.3 (GND), LMP7721.2 (N/C_2), LMP7721.3, LMP7721.5 (N/C_5), LMP7721.7 (N/C_7), OPA2320_1.4 (V-), OPA2320_2.4 (V-), OSD5-5D1.2 (A), R11.1, TLV333.2 (V_)
- net at R8.1, R9.2: now also DAC7571.6 (A0)
- net at R8.2: now also DAC7571.3 (VDD)
- net at C7.1, R6.1: now also LMP7721.8, OSD5-5D1.1 (K)
- new net: OPA2320_1.3 (+INA), OPA2320_1.5 (+INB)
- new net: JWF1.1 (IN), R11.2
- new net VCC: JWF1.2 (V+)
- new net jwf_5: JWF1.5 (COM), R10.1
